Commit message: added realsense octomap

File: src/openarm_description/urdf/robot/v10.urdf.xacro (robot description, xacro)
@@ -61,3 +61,7 @@
   can_fd="$(arg can_fd)"
   />
+  <xacro:include filename="$(find realsense2_description)/urdf/_d455.urdf.xacro" />
+  <xacro:sensor_d455 parent="world" name="camera">
+    <origin xyz="0.100 0.000 0.735" rpy="0 1.0472 0"/>
+  </xacro:sensor_d455>
 </robot>

Commit message: changes made

File: src/openarm_description/urdf/robot/v10.urdf.xacro (robot description, xacro)
@@ -63,5 +63,6 @@
   <xacro:include filename="$(find realsense2_description)/urdf/_d455.urdf.xacro" />
   <xacro:sensor_d455 parent="world" name="camera">
-    <origin xyz="0.100 0.000 0.735" rpy="0 1.0472 0"/>
+    <!-- Measured camera mount position; retain verified +60 deg ROS pitch. -->
+    <origin xyz="0.16089 0.000 0.72846" rpy="0 1.0472 0"/>
   </xacro:sensor_d455>
 </robot>

Commit message: Added VLM scripts and camera corrected

File: src/openarm_description/urdf/robot/v10.urdf.xacro (robot description, xacro)
@@ -64,5 +64,5 @@
   <xacro:sensor_d455 parent="world" name="camera">
     <!-- Measured camera mount position; retain verified +60 deg ROS pitch. -->
-    <origin xyz="0.16089 0.000 0.72846" rpy="0 1.0472 0"/>
+    <origin xyz="0.10175 0.000 0.99272" rpy="0 1.0472 0"/>
   </xacro:sensor_d455>
 </robot>
