Commit message: left and right decision making

File: openarm.urdf (robot description, URDF)
Before this commit: robot openarm, 26 links, 25 joints
Joints:
- joint openarm_left_joint4: limit lower=0.0 upper=2.443461 effort=27 velocity=5.445426 -> lower=-0.05 upper=2.443461 effort=27 velocity=5.445426
- joint openarm_right_joint4: limit lower=0.0 upper=2.443461 effort=27 velocity=5.445426 -> lower=-0.05 upper=2.443461 effort=27 velocity=5.445426

Commit message: edited GraspModel GenX

File: openarm.urdf (robot description, URDF)
Before this commit: robot openarm, 26 links, 25 joints
Joints:
- joint openarm_left_finger_joint2: limit lower=0.0 upper=0.044 effort=333 velocity=10.0 -> lower=-0.030 upper=0.044 effort=333 velocity=10.0
- joint openarm_right_finger_joint2: limit lower=0.0 upper=0.044 effort=333 velocity=10.0 -> lower=-0.030 upper=0.044 effort=333 velocity=10.0

File: src/openarm_description/urdf/ee/openarm_hand.xacro (robot description, xacro)
@@ -67,5 +67,14 @@
       <origin xyz="0 0.006 0.015" rpy="0 0 0" />
       <axis xyz="0 1 0" />
-      <limit effort="333" lower="0.0" upper="0.044" velocity="10.0" />
+      <!-- Lower bound matches finger_joint1's, because this joint mimics it
+           with multiplier 1 and offset 0: whatever joint1 is commanded to,
+           this one is required to follow exactly. With lower="0.0" the pair
+           was inconsistent - joint1 could be driven to -0.030 while this
+           joint's floor was 0 - and cuRobo refuses to build a kinematic
+           model from it: "mimic joint can go out of it's lower limit as
+           active joint has larger range". That refusal is why the fingers
+           could not be given collision spheres, and the fingers are exactly
+           the links that were driving through the torso unchecked. -->
+      <limit effort="333" lower="-0.030" upper="0.044" velocity="10.0" />
       <mimic joint="${ee_prefix}finger_joint1" />
     </joint>

Commit message: changes made

File: openarm.urdf (robot description, URDF)
Before this commit: robot openarm, 26 links, 25 joints
Joints:
- joint openarm_left_openarm_body_link0_joint: origin xyz=0.0 0.051 0.698 rpy=-1.5708 0 0 -> xyz=0.0126 0.0572 0.7344 rpy=-1.5708 0 0
- joint openarm_right_openarm_body_link0_joint: origin xyz=0.0 -0.051 0.698 rpy=1.5708 0 0 -> xyz=0.0126 -0.0448 0.7344 rpy=1.5708 0 0

File: src/openarm_description/urdf/robot/v10.urdf.xacro (robot description, xacro)
@@ -22,7 +22,10 @@
   <xacro:arg name="fake_sensor_commands" default="false" />
   <xacro:arg name="bimanual" default="false" />
-  <xacro:arg name="right_arm_base_xyz" default="0.0 -0.051 0.698" />
+  <!-- V7 (2026-10-06): arm mount moved by (+12.6, +6.2, +36.4) mm so that the
+       camera can sit at its tape-measured position (V4) and still agree with what it
+       sees of the arms (CALIBRATE, 24 poses). Was 0.0 -/+0.051 0.698. See cam_org.txt. -->
+  <xacro:arg name="right_arm_base_xyz" default="0.0126 -0.0448 0.7344" />
   <xacro:arg name="right_arm_base_rpy" default="1.5708 0 0" />
-  <xacro:arg name="left_arm_base_xyz" default="0.0 0.051 0.698" />
+  <xacro:arg name="left_arm_base_xyz" default="0.0126 0.0572 0.7344" />
   <xacro:arg name="left_arm_base_rpy" default="-1.5708 0 0" />
   <xacro:arg name="can_fd" default="true" />
@@ -63,6 +66,7 @@
   <xacro:include filename="$(find realsense2_description)/urdf/_d455.urdf.xacro" />
   <xacro:sensor_d455 parent="world" name="camera">
-    <!-- Measured camera mount position; retain verified +60 deg ROS pitch. -->
-    <origin xyz="0.10175 0.000 0.99272" rpy="0 1.0472 0"/>
+    <!-- V7: the V4 tape position, orientation fine-tuned by CALIBRATE (the arms were
+         moved instead, see right_arm_base_xyz). History in cam_org.txt. -->
+    <origin xyz="0.01233 0.000 0.53131" rpy="0.02056 -0.07726 -0.01912"/>
   </xacro:sensor_d455>
 </robot>

Commit message: pick with new model

File: openarm.urdf (robot description, URDF)
Before this commit: robot openarm, 26 links, 25 joints
Links:
- link openarm_left_hand: geometry collision cylinder length=0.0954 radius=0.015; visual cylinder length=0.13815 radius=0.015
- link openarm_left_left_finger: geometry 
- link openarm_left_link7: geometry collision cylinder length=0.1001 radius=0.015; visual cylinder length=0.1001 radius=0.015
- link openarm_left_right_finger: geometry 

File: src/openarm_description/urdf/arm/openarm_arm.xacro (robot description, xacro)
@@ -74,5 +74,28 @@
       <xacro:openarm-limits name="joint6" config="${joint_limits}" />
     </joint>
-    <xacro:link_with_sc no_prefix="${no_prefix}" name="link7" kinematics_link="${kinematics_link}" inertials="${inertials}" reflect="${reflect}"/>
+    <!-- link7: the LEFT arm's wrist shell is replaced by a plain cylinder,
+         30 mm across, from joint 7 to the hand mount (100.1 mm, unchanged);
+         joint 7 still turns it (2026-10-26). The right arm keeps its mesh. -->
+    <xacro:if value="${arm_prefix == 'left_'}">
+      <link name="${prefix}link7">
+        <visual name="${prefix}link7_visual">
+          <origin rpy="0 0 0" xyz="0 0 0.05005"/>
+          <geometry>
+            <cylinder radius="0.015" length="0.1001"/>
+          </geometry>
+          <material name="grey"><color rgba="0.6 0.6 0.62 1.0"/></material>
+        </visual>
+        <collision name="${prefix}link7_collision">
+          <origin rpy="0 0 0" xyz="0 0 0.05005"/>
+          <geometry>
+            <cylinder radius="0.015" length="0.1001"/>
+          </geometry>
+        </collision>
+        <xacro:openarm-inertials name="link7" inertials="${inertials}" reflect="${reflect}" />
+      </link>
+    </xacro:if>
+    <xacro:unless value="${arm_prefix == 'left_'}">
+      <xacro:link_with_sc no_prefix="${no_prefix}" name="link7" kinematics_link="${kinematics_link}" inertials="${inertials}" reflect="${reflect}"/>
+    </xacro:unless>
     <joint name="${prefix}joint7" type="revolute">
       <xacro:openarm-kinematics name="joint7" config="${kinematics}" />

File: src/openarm_description/urdf/ee/openarm_hand.xacro (robot description, xacro)
@@ -8,5 +8,32 @@
       <xacro:property name="ee_prefix" value="openarm_${arm_prefix}" />
     </xacro:unless>
-    <xacro:ee_link_with_sc name="hand" prefix="${ee_prefix}" ee_kinematics_link="${ee_kinematics_link}"/>
+    <!-- The LEFT gripper is a plain grey cylinder, 30 mm across, 138.15 mm from
+         the hand mount: 238.25 mm from joint 7, measured, to the working tip
+         (2026-10-26); no fingers. Its collision shape stops at 95.4 mm (the
+         old fingertips): the last 42.75 mm is the tool's collision piece
+         (tools.yaml, ctm/robot.py), which alone may touch at the contact. The
+         finger links and joints stay, without shapes, so the controllers and
+         planners keep the same joints. The right gripper is unchanged. -->
+    <xacro:if value="${arm_prefix == 'left_'}">
+      <link name="${ee_prefix}hand">
+        <visual name="${ee_prefix}hand_visual">
+          <origin rpy="0 0 0" xyz="0 0 0.069075"/>
+          <geometry>
+            <cylinder radius="0.015" length="0.13815"/>
+          </geometry>
+          <material name="grey"><color rgba="0.6 0.6 0.62 1.0"/></material>
+        </visual>
+        <collision name="${ee_prefix}hand_collision">
+          <origin rpy="0 0 0" xyz="0 0 0.0477"/>
+          <geometry>
+            <cylinder radius="0.015" length="0.0954"/>
+          </geometry>
+        </collision>
+        <xacro:ee-inertials name="hand" />
+      </link>
+    </xacro:if>
+    <xacro:unless value="${arm_prefix == 'left_'}">
+      <xacro:ee_link_with_sc name="hand" prefix="${ee_prefix}" ee_kinematics_link="${ee_kinematics_link}"/>
+    </xacro:unless>
     <!-- <link name="${ee_prefix}hand"/> -->
     <xacro:unless value="${connected_to == ''}">
@@ -25,4 +52,13 @@
       <child link="${ee_prefix}hand_tcp" />
     </joint>
+    <xacro:if value="${arm_prefix == 'left_'}">
+      <link name="${ee_prefix}left_finger">
+        <xacro:ee-inertials name="left_finger"/>
+      </link>
+      <link name="${ee_prefix}right_finger">
+        <xacro:ee-inertials name="right_finger"/>
+      </link>
+    </xacro:if>
+    <xacro:unless value="${arm_prefix == 'left_'}">
     <link name="${ee_prefix}left_finger">
       <visual name="${ee_prefix}left_finger_visual">
@@ -55,4 +91,5 @@
       <xacro:ee-inertials name="right_finger"/>
     </link>
+    </xacro:unless>
     <joint name="${ee_prefix}finger_joint1" type="prismatic">
       <parent link="${ee_prefix}hand" />
